Commit message: feat: add LiDAR and SLAM mapping pipeline

File: ros_ws/src/serving_robot_description/urdf/sensors.xacro (robot description, xacro)
@@ -1,13 +1,78 @@
 <?xml version="1.0"?>
 <robot xmlns:xacro="http://www.ros.org/wiki/xacro">
-  <xacro:macro name="serving_robot_sensors" params="">
-    <!--
-      Sensors are intentionally added in M2.
-      Planned frames:
-        laser_link
-        camera_link
-        camera_color_optical_frame
-        camera_depth_optical_frame
-    -->
+  <xacro:macro
+    name="serving_robot_sensors"
+    params="robot_name">
+    <!-- ======================================================= -->
+    <!-- 2D LiDAR                                                 -->
+    <!-- ======================================================= -->
+    <link name="laser_link">
+      <visual>
+        <origin xyz="0 0 0" rpy="0 0 0"/>
+        <geometry>
+          <cylinder
+            radius="0.035"
+            length="0.04"/>
+        </geometry>
+        <material name="lidar_black">
+          <color rgba="0.03 0.03 0.03 1.0"/>
+        </material>
+      </visual>
+      <collision>
+        <origin xyz="0 0 0" rpy="0 0 0"/>
+        <geometry>
+          <cylinder
+            radius="0.035"
+            length="0.04"/>
+        </geometry>
+      </collision>
+      <inertial>
+        <origin xyz="0 0 0" rpy="0 0 0"/>
+        <mass value="0.15"/>
+        <inertia
+          ixx="0.000066"
+          ixy="0.0"
+          ixz="0.0"
+          iyy="0.000066"
+          iyz="0.0"
+          izz="0.000092"/>
+      </inertial>
+    </link>
+    <joint name="laser_joint" type="fixed">
+      <parent link="base_link"/>
+      <child link="laser_link"/>
+      <origin
+        xyz="0 0 0.18"
+        rpy="0 0 0"/>
+    </joint>
+    <!-- ======================================================= -->
+    <!-- Gazebo Harmonic GPU LiDAR                               -->
+    <!-- ======================================================= -->
+    <gazebo reference="laser_link">
+      <sensor
+        name="gpu_lidar"
+        type="gpu_lidar">
+        <always_on>true</always_on>
+        <visualize>true</visualize>
+        <update_rate>10</update_rate>
+        <topic>/model/${robot_name}/scan</topic>
+        <gz_frame_id>laser_link</gz_frame_id>
+        <lidar>
+          <scan>
+            <horizontal>
+              <samples>720</samples>
+              <resolution>1</resolution>
+              <min_angle>-3.14159265359</min_angle>
+              <max_angle>3.14159265359</max_angle>
+            </horizontal>
+          </scan>
+          <range>
+            <min>0.10</min>
+            <max>12.0</max>
+            <resolution>0.01</resolution>
+          </range>
+        </lidar>
+      </sensor>
+    </gazebo>
   </xacro:macro>
 </robot>

File: ros_ws/src/serving_robot_description/urdf/serving_robot.urdf.xacro (robot description, xacro)
@@ -3,4 +3,7 @@
   xmlns:xacro="http://www.ros.org/wiki/xacro"
   name="serving_robot">
+  <xacro:arg
+    name="robot_name"
+    default="robot_01"/>
   <xacro:include
     filename="$(find serving_robot_description)/urdf/base.xacro"/>
@@ -8,4 +11,5 @@
     filename="$(find serving_robot_description)/urdf/sensors.xacro"/>
   <xacro:serving_robot_base/>
-  <xacro:serving_robot_sensors/>
+  <xacro:serving_robot_sensors
+    robot_name="$(arg robot_name)"/>
 </robot>
